Commit message: BIg update with camera intrinsics and extrisnics and should cleaned up on monday

File: ur_gripper_control/urdf/ur_gripper_controlled.urdf.xacro (robot description, xacro)
@@ -6,10 +6,10 @@
   <xacro:include filename="$(find ur_robot_driver)/urdf/ur.ros2_control.xacro"/>
   <!--We need to specify the arguments used for parametrizing our description-->
-  <xacro:arg name="ur_type" default="ur5e"/>
+  <xacro:arg name="ur_type" default="ur10"/>
   <xacro:arg name="joint_limit_parameters_file" default="$(find ur_description)/config/$(arg ur_type)/joint_limits.yaml"/>
   <xacro:arg name="kinematics_parameters_file" default="$(find ur_description)/config/$(arg ur_type)/default_kinematics.yaml"/>
   <xacro:arg name="physical_parameters_file" default="$(find ur_description)/config/$(arg ur_type)/physical_parameters.yaml"/>
   <xacro:arg name="visual_parameters_file" default="$(find ur_description)/config/$(arg ur_type)/visual_parameters.yaml"/>
-  <xacro:arg name="robot_ip" default="0.0.0.0"/>
+  <xacro:arg name="robot_ip" default="192.168.1.2"/>
   <xacro:arg name="headless_mode" default="false" />
   <xacro:arg name="ur_script_filename" default="$(find ur_client_library)/resources/external_control.urscript"/>

File: ur_gripper_description/urdf/ur_gripper.urdf.xacro (robot description, xacro)
@@ -2,5 +2,5 @@
 <robot name="ur_gripper" xmlns:xacro="http://ros.org/wiki/xacro">
   <xacro:include filename="$(find ur_gripper_description)/urdf/ur_gripper_macro.xacro"/>
-  <xacro:arg name="ur_type" default="ur5e"/>
+  <xacro:arg name="ur_type" default="ur10"/>
   <xacro:arg name="joint_limits_parameters_file" default="$(find ur_description)/config/$(arg ur_type)/joint_limits.yaml"/>
   <xacro:arg name="kinematics_parameters_file" default="$(find ur_description)/config/$(arg ur_type)/default_kinematics.yaml"/>

File: ur_gripper_description/urdf/ur_gripper_macro.xacro (robot description, xacro)
@@ -12,8 +12,68 @@
     ">
     <link name="robot_base"/>
-    <joint name="base_joint" type="fixed">
-      <xacro:insert_block name="origin" />
-      <parent link="${parent}" />
-      <child link="robot_base" />
+    <!-- Table base (dimensions 120x80x20 cm) -->
+    <link name="table_base">
+      <visual>
+        <geometry>
+          <box size="1.2 0.8 0.2"/>
+        </geometry>
+        <origin rpy="0 0 0" xyz="0 0 0.1"/> <!-- Center of the base -->
+        <material name="grey">
+          <color rgba="0.7 0.7 0.7 1.0"/>
+        </material>
+      </visual>
+      <collision>
+        <geometry>
+          <box size="1.2 0.8 0.2"/>
+        </geometry>
+        <origin rpy="0 0 0" xyz="0 0 0.1"/>
+      </collision>
+      <inertial> <!-- Add inertial properties -->
+        <mass value="50"/>
+        <inertia ixx="2.7" ixy="0.0" ixz="0.0" iyy="4.0" iyz="0.0" izz="5.3"/>
+      </inertial>
+    </link>
+    <!-- Joint to connect the table base to the world -->
+    <joint name="world_to_table_base" type="fixed">
+      <parent link="${parent}"/>
+      <child link="table_base"/>
+      <origin xyz="0 0 0" rpy="0 0 0"/>
+    </joint>
+    <!-- Table (dimensions 100x40x72 cm) -->
+    <link name="table">
+      <visual>
+        <geometry>
+          <box size="1.0 0.40 0.72"/>
+        </geometry>
+        <origin rpy="0 0 0" xyz="0 0 0.36"/> <!-- Center of the table -->
+        <material name="brown">
+          <color rgba="0.8 0.6 0.4 1.0"/>
+        </material>
+      </visual>
+      <collision>
+        <geometry>
+          <box size="1.0 0.40 0.72"/>
+        </geometry>
+        <origin rpy="0 0 0" xyz="0 0 0.36"/>
+      </collision>
+      <inertial> <!-- Add inertial properties -->
+        <mass value="20"/>
+        <inertia ixx="1.0" ixy="0.0" ixz="0.0" iyy="1.2" iyz="0.0" izz="0.8"/>
+      </inertial>
+    </link>
+    <!-- Joint to connect the table to the table base -->
+    <joint name="table_base_to_table" type="fixed">
+      <parent link="table_base"/>
+      <child link="table"/>
+      <!-- Position the table on top of the table base -->
+      <origin xyz="0.1 0 0.2" rpy="0 0 0"/>
+    </joint>
+    <!-- Important: Connect robot base to the table instead of world -->
+    <joint name="table_to_robot_base" type="fixed">
+      <parent link="table"/>
+      <child link="robot_base"/>
+      <!-- Position the robot on top of the table surface -->
+      <!-- 0.36 (to table center) + 0.36 (half table height) = 0.72 (to table top) -->
+      <origin xyz="-0.3 0.025 0.72" rpy="0 0 3.1419"/>
     </joint>
     <!--This will create the specific robot-->

File: ur_gripper_moveit_config/config/ur_gripper.ros2_control.xacro (robot description, xacro)
@@ -8,43 +8,43 @@
                 <plugin>mock_components/GenericSystem</plugin>
             </hardware>
-            <joint name="ur5e_shoulder_pan_joint">
+            <joint name="ur10_shoulder_pan_joint">
                 <command_interface name="position"/>
                 <state_interface name="position">
-                  <param name="initial_value">${initial_positions['ur5e_shoulder_pan_joint']}</param>
+                  <param name="initial_value">${initial_positions['ur10_shoulder_pan_joint']}</param>
                 </state_interface>
                 <state_interface name="velocity"/>
             </joint>
-            <joint name="ur5e_shoulder_lift_joint">
+            <joint name="ur10_shoulder_lift_joint">
                 <command_interface name="position"/>
                 <state_interface name="position">
-                  <param name="initial_value">${initial_positions['ur5e_shoulder_lift_joint']}</param>
+                  <param name="initial_value">${initial_positions['ur10_shoulder_lift_joint']}</param>
                 </state_interface>
                 <state_interface name="velocity"/>
             </joint>
-            <joint name="ur5e_elbow_joint">
+            <joint name="ur10_elbow_joint">
                 <command_interface name="position"/>
                 <state_interface name="position">
-                  <param name="initial_value">${initial_positions['ur5e_elbow_joint']}</param>
+                  <param name="initial_value">${initial_positions['ur10_elbow_joint']}</param>
                 </state_interface>
                 <state_interface name="velocity"/>
             </joint>
-            <joint name="ur5e_wrist_1_joint">
+            <joint name="ur10_wrist_1_joint">
                 <command_interface name="position"/>
                 <state_interface name="position">
-                  <param name="initial_value">${initial_positions['ur5e_wrist_1_joint']}</param>
+                  <param name="initial_value">${initial_positions['ur10_wrist_1_joint']}</param>
                 </state_interface>
                 <state_interface name="velocity"/>
             </joint>
-            <joint name="ur5e_wrist_2_joint">
+            <joint name="ur10_wrist_2_joint">
                 <command_interface name="position"/>
                 <state_interface name="position">
-                  <param name="initial_value">${initial_positions['ur5e_wrist_2_joint']}</param>
+                  <param name="initial_value">${initial_positions['ur10_wrist_2_joint']}</param>
                 </state_interface>
                 <state_interface name="velocity"/>
             </joint>
-            <joint name="ur5e_wrist_3_joint">
+            <joint name="ur10_wrist_3_joint">
                 <command_interface name="position"/>
                 <state_interface name="position">
-                  <param name="initial_value">${initial_positions['ur5e_wrist_3_joint']}</param>
+                  <param name="initial_value">${initial_positions['ur10_wrist_3_joint']}</param>
                 </state_interface>
                 <state_interface name="velocity"/>
