Commit message: ur10_moveit_config almost ready and extrisnic camera calirbtation

File: ur_gripper_description/urdf/ur_gripper_macro.xacro (robot description, xacro)
@@ -75,5 +75,5 @@
       <!-- Position the robot on top of the table surface -->
       <!-- 0.36 (to table center) + 0.36 (half table height) = 0.72 (to table top) -->
-      <origin xyz="-0.3 0.025 0.72" rpy="0 0 3.1419"/>
+      <origin xyz="-0.3 0.025 0.76" rpy="0 0 3.0543"/>  <!-- 3.1419 - (5 * π/180) = 3.0543 -->
     </joint>
     <!--This will create the specific robot-->
@@ -110,4 +110,96 @@
       <origin xyz="0 0 0" rpy="0 0 0"/>
     </joint>
+    <!-- Add a RealSense D455 camera -->
+    <link name="camera_link">
+      <visual>
+        <geometry>
+         <box size="0.035 0.09 0.035"/>
+        </geometry>
+        <material name="aluminum">
+          <color rgba="0.5 0.5 0.5 1.0"/>
+        </material>
+      </visual>
+      <collision>
+        <geometry>
+          <box size="0.035 0.09 0.035"/>
+        </geometry>
+      </collision>
+      <inertial>
+        <mass value="0.072"/>
+        <inertia ixx="0.00006" ixy="0" ixz="0" iyy="0.00006" iyz="0" izz="0.00006"/>
+      </inertial>
+    </link>
+    <!-- Camera mount structure -->
+    <link name="camera_mount_horizontal">
+      <visual>
+        <origin xyz="0 0 -0.3" rpy="0 0 0"/> <!-- Extend 60cm backward in camera frame -->
+        <geometry>
+          <box size="0.02 0.02 0.6"/>
+        </geometry>
+        <material name="dark_aluminum">
+          <color rgba="0.4 0.4 0.4 1.0"/>
+        </material>
+      </visual>
+      <collision>
+        <origin xyz="0 0 -0.3" rpy="0 0 0"/>
+        <geometry>
+          <box size="0.02 0.02 0.6"/>
+        </geometry>
+      </collision>
+      <inertial>
+        <mass value="0.5"/>
+        <inertia ixx="0.001" ixy="0" ixz="0" iyy="0.001" iyz="0" izz="0.015"/>
+      </inertial>
+    </link>
+    <!-- Replace the camera_mount_vertical link and joint -->
+    <link name="camera_mount_vertical">
+      <visual>
+        <!-- Change from x-direction to z-direction for downward orientation -->
+        <origin xyz="0 0 -1.05" rpy="0 0 0"/> <!-- Extend 210cm downward -->
+        <geometry>
+          <box size="0.02 0.02 2.1"/>
+        </geometry>
+        <material name="dark_aluminum">
+          <color rgba="0.4 0.4 0.4 1.0"/>
+        </material>
+      </visual>
+      <collision>
+        <origin xyz="0 0 -1.05" rpy="0 0 0"/>
+        <geometry>
+          <box size="0.02 0.02 2.1"/>
+        </geometry>
+      </collision>
+      <inertial>
+        <mass value="1.0"/>
+        <inertia ixx="0.04" ixy="0" ixz="0" iyy="0.04" iyz="0" izz="0.001"/>
+      </inertial>
+    </link>
+    <!-- Connect horizontal to vertical mount -->
+    <joint name="mount_horizontal_to_vertical" type="fixed">
+      <parent link="camera_mount_horizontal"/>
+      <child link="camera_mount_vertical"/>
+      <!-- Position at the end of the horizontal beam and rotate 90 degrees around Y to point downward -->
+      <origin xyz="0 0.03 -0.6" rpy="0 -1.5708 0"/>
+    </joint>
+    <!-- Connect camera to horizontal mount -->
+    <joint name="camera_to_mount_horizontal" type="fixed">
+      <parent link="camera_link"/>
+      <child link="camera_mount_horizontal"/>
+      <!-- Attach to the back center of the camera -->
+      <origin xyz="0 0 -0.02" rpy="0 0 0"/>
+    </joint>
+    <!-- Connect camera to the robot's base link -->
+    <joint name="ur10_base_link_to_camera" type="fixed">
+      <parent link="${ur_type}_base_link"/>
+      <child link="camera_link"/>
+      <origin xyz="0.440200 0.059500 1.112700" rpy="-2.4667 1.55676 -0.8047"/>
+    </joint>
+    <!-- Add TCP frame -->
+    <link name="${ur_type}_tcp"/>
+    <joint name="tool0_to_tcp" type="fixed">
+      <parent link="${ur_type}_tool0"/>
+      <child link="${ur_type}_tcp"/>
+      <origin xyz="0 0 0.11" rpy="0 0 0"/>
+    </joint>
   </xacro:macro>
 </robot>

Commit message: gripper interface and node ready

File: ur_gripper_description/urdf/ur_gripper_macro.xacro (robot description, xacro)
@@ -44,7 +44,7 @@
       <visual>
         <geometry>
-          <box size="1.0 0.40 0.72"/>
-        </geometry>
-        <origin rpy="0 0 0" xyz="0 0 0.36"/> <!-- Center of the table -->
+          <box size="1.0 0.40 0.76"/>
+        </geometry>
+        <origin rpy="0 0 0" xyz="0 0 0.38"/> <!-- Center of the table -->
         <material name="brown">
           <color rgba="0.8 0.6 0.4 1.0"/>
@@ -53,7 +53,7 @@
       <collision>
         <geometry>
-          <box size="1.0 0.40 0.72"/>
-        </geometry>
-        <origin rpy="0 0 0" xyz="0 0 0.36"/>
+          <box size="1.0 0.40 0.76"/>
+        </geometry>
+        <origin rpy="0 0 0" xyz="0 0 0.38"/>
       </collision>
       <inertial> <!-- Add inertial properties -->
@@ -89,4 +89,23 @@
       <origin xyz="0 0 0" rpy="0 0 0" />
     </xacro:ur_robot>
+    <link name="quick_tool_changer">
+      <visual>
+        <origin xyz="0 0 0" rpy="${-pi/2} ${0} ${0}"/>
+        <geometry>
+          <mesh filename="package://ur_gripper_description/meshes/quick_changer.dae" scale="0.001 0.001 0.001"/>
+        </geometry>
+        </visual>
+        <collision>
+          <origin xyz="0 0 0" rpy="${0} ${0} ${0}"/>
+          <geometry>
+          <box size="0.09 0.09 0.016"/>
+          </geometry>
+        </collision>
+        </link>
+    <joint name="tool0_to_quick_tool_changer" type="fixed">
+      <parent link="${ur_type}_tool0"/>
+      <child link="quick_tool_changer"/>
+      <origin xyz="0 0 0" rpy="0 0 0"/>
+    </joint>
     <!-- Add a simple gripper -->
     <link name="gripper">
@@ -94,11 +113,11 @@
         <origin xyz="0 0 0" rpy="${-pi/2} ${0} ${0}"/>
         <geometry>
-          <mesh filename="package://ur_gripper_description/meshes/VacuumGripper.dae" scale="0.001 0.001 0.001"/>
-        </geometry>
-      </visual>
-      <collision>
-        <origin xyz="0.0 0 0.05" rpy="${0} ${0} ${0}"/>
-        <geometry>
-          <box size="0.14 0.14 0.1"/>
+          <mesh filename="package://ur_gripper_description/meshes/VG10_v2.dae" scale="0.001 0.001 0.001"/>
+        </geometry>
+      </visual>
+      <collision>
+        <origin xyz="0.0 0 0.066" rpy="${0} ${0} ${0}"/>
+        <geometry>
+          <box size="0.15 0.15 0.11"/>
         </geometry>
       </collision>
@@ -106,5 +125,5 @@
     <!-- Connect gripper to the robot's end effector -->
     <joint name="tool0_to_gripper" type="fixed">
-      <parent link="${ur_type}_tool0"/>
+      <parent link="quick_tool_changer"/>
       <child link="gripper"/>
       <origin xyz="0 0 0" rpy="0 0 0"/>

Commit message: cartesian path for mtc and image processor node modification

File: ur_gripper_description/urdf/ur_gripper_macro.xacro (robot description, xacro)
@@ -97,5 +97,5 @@
         </visual>
         <collision>
-          <origin xyz="0 0 0" rpy="${0} ${0} ${0}"/>
+          <origin xyz="0 0 0.008" rpy="${0} ${0} ${0}"/>
           <geometry>
           <box size="0.09 0.09 0.016"/>
@@ -152,7 +152,7 @@
     <link name="camera_mount_horizontal">
       <visual>
-        <origin xyz="0 0 -0.3" rpy="0 0 0"/> <!-- Extend 60cm backward in camera frame -->
-        <geometry>
-          <box size="0.02 0.02 0.6"/>
+        <origin xyz="0 0 -0.225" rpy="0 0 0"/> <!-- Extend 60cm backward in camera frame -->
+        <geometry>
+          <box size="0.02 0.02 0.45"/>
         </geometry>
         <material name="dark_aluminum">
@@ -161,7 +161,7 @@
       </visual>
       <collision>
-        <origin xyz="0 0 -0.3" rpy="0 0 0"/>
-        <geometry>
-          <box size="0.02 0.02 0.6"/>
+        <origin xyz="0 0 -0.225" rpy="0 0 0"/>
+        <geometry>
+          <box size="0.02 0.02 0.45"/>
         </geometry>
       </collision>
@@ -177,5 +177,5 @@
         <origin xyz="0 0 -1.05" rpy="0 0 0"/> <!-- Extend 210cm downward -->
         <geometry>
-          <box size="0.02 0.02 2.1"/>
+          <box size="0.03 0.03 2.1"/>
         </geometry>
         <material name="dark_aluminum">
@@ -186,5 +186,5 @@
         <origin xyz="0 0 -1.05" rpy="0 0 0"/>
         <geometry>
-          <box size="0.02 0.02 2.1"/>
+          <box size="0.03 0.03 2.1"/>
         </geometry>
       </collision>
@@ -199,5 +199,5 @@
       <child link="camera_mount_vertical"/>
       <!-- Position at the end of the horizontal beam and rotate 90 degrees around Y to point downward -->
-      <origin xyz="0 0.03 -0.6" rpy="0 -1.5708 0"/>
+      <origin xyz="0 0.03 -0.45" rpy="0 -1.5708 0"/>
     </joint>
     <!-- Connect camera to horizontal mount -->
@@ -219,5 +219,5 @@
       <parent link="${ur_type}_tool0"/>
       <child link="${ur_type}_tcp"/>
-      <origin xyz="0 0 0.11" rpy="0 0 0"/>
+      <origin xyz="0 0 0.126" rpy="0 0 0"/>
     </joint>
     <!-- Add a virtual vacuum gripper control link and joint -->
